File: 2U-NTP-Clock.kicad_pcb (KiCad board)
At the start: 2 copper layers, 0 parts

Commit message: 基板外形作成
Other:
- board outline added: 482.6 x 83.8 mm

Commit message: 回路図作成
Parts:
- added U1: ~, stamp:STAMP-S3-DIP, F.Cu at (114.3, 229.9)
- added U2: ~, TinyRTC:TinyRTC_Battery_Side_Up, F.Cu at (114.3, 177.8)
Routing:
- net SQ: track 0.00 -> 74.3 mm
- net SCL: track 0.00 -> 69.4 mm
- net SDA: track 0.00 -> 64.3 mm

Commit message: トランジスタ以外配置した
Parts:
- added D1: LED, LED_THT:LED_D5.0mm, F.Cu at (149.9, 165.1)
- added D10: LED, LED_THT:LED_D5.0mm, F.Cu at (176.5, 219.7)
- added D100: LED, LED_THT:LED_D5.0mm, F.Cu at (341.6, 241.3)
- added D101: LED, LED_THT:LED_D5.0mm, F.Cu at (311.1, 210.8)
- added D102: LED, LED_THT:LED_D5.0mm, F.Cu at (309.9, 219.7)
- added D103: LED, LED_THT:LED_D5.0mm, F.Cu at (308.6, 228.6)
- added D104: LED, LED_THT:LED_D5.0mm, F.Cu at (307.3, 237.5)
- added D105: LED, LED_THT:LED_D5.0mm, F.Cu at (315.0, 171.4)
- added D106: LED, LED_THT:LED_D5.0mm, F.Cu at (313.7, 180.3)
- added D107: LED, LED_THT:LED_D5.0mm, F.Cu at (312.4, 189.2)
- added D108: LED, LED_THT:LED_D5.0mm, F.Cu at (311.1, 198.1)
- added D109: LED, LED_THT:LED_D5.0mm, F.Cu at (318.8, 203.2)
- added D11: LED, LED_THT:LED_D5.0mm, F.Cu at (175.3, 228.6)
- added D110: LED, LED_THT:LED_D5.0mm, F.Cu at (327.7, 203.2)
- added D111: LED, LED_THT:LED_D5.0mm, F.Cu at (336.6, 203.2)
- added D112: LED, LED_THT:LED_D5.0mm, F.Cu at (345.4, 203.2)
- added D113: LED, LED_THT:LED_D5.0mm, F.Cu at (391.2, 165.1)
- added D114: LED, LED_THT:LED_D5.0mm, F.Cu at (400.1, 165.1)
- added D115: LED, LED_THT:LED_D5.0mm, F.Cu at (408.9, 165.1)
- added D116: LED, LED_THT:LED_D5.0mm, F.Cu at (417.8, 165.1)
- added D117: LED, LED_THT:LED_D5.0mm, F.Cu at (422.9, 171.4)
- added D118: LED, LED_THT:LED_D5.0mm, F.Cu at (421.6, 180.3)
- added D119: LED, LED_THT:LED_D5.0mm, F.Cu at (420.4, 189.2)
- added D12: LED, LED_THT:LED_D5.0mm, F.Cu at (174.0, 237.5)
- added D120: LED, LED_THT:LED_D5.0mm, F.Cu at (419.1, 198.1)
- added D121: LED, LED_THT:LED_D5.0mm, F.Cu at (419.1, 210.8)
- added D122: LED, LED_THT:LED_D5.0mm, F.Cu at (417.8, 219.7)
- added D123: LED, LED_THT:LED_D5.0mm, F.Cu at (416.6, 228.6)
- added D124: LED, LED_THT:LED_D5.0mm, F.Cu at (415.3, 237.5)
- added D125: LED, LED_THT:LED_D5.0mm, F.Cu at (383.5, 241.3)
- added D126: LED, LED_THT:LED_D5.0mm, F.Cu at (392.4, 241.3)
- added D127: LED, LED_THT:LED_D5.0mm, F.Cu at (401.3, 241.3)
- added D128: LED, LED_THT:LED_D5.0mm, F.Cu at (410.2, 241.3)
- added D129: LED, LED_THT:LED_D5.0mm, F.Cu at (379.7, 210.8)
- added D13: LED, LED_THT:LED_D5.0mm, F.Cu at (142.2, 241.3)
- added D130: LED, LED_THT:LED_D5.0mm, F.Cu at (378.5, 219.7)
- added D131: LED, LED_THT:LED_D5.0mm, F.Cu at (377.2, 228.6)
- added D132: LED, LED_THT:LED_D5.0mm, F.Cu at (375.9, 237.5)
- added D133: LED, LED_THT:LED_D5.0mm, F.Cu at (383.5, 171.4)
- added D134: LED, LED_THT:LED_D5.0mm, F.Cu at (382.3, 180.3)
- added D135: LED, LED_THT:LED_D5.0mm, F.Cu at (381.0, 189.2)
- added D136: LED, LED_THT:LED_D5.0mm, F.Cu at (379.7, 198.1)
- added D137: LED, LED_THT:LED_D5.0mm, F.Cu at (387.4, 203.2)
- added D138: LED, LED_THT:LED_D5.0mm, F.Cu at (396.2, 203.2)
- added D139: LED, LED_THT:LED_D5.0mm, F.Cu at (405.1, 203.2)
- added D14: LED, LED_THT:LED_D5.0mm, F.Cu at (151.1, 241.3)
- added D140: LED, LED_THT:LED_D5.0mm, F.Cu at (414.0, 203.2)
- added D141: LED, LED_THT:LED_D5.0mm, F.Cu at (443.2, 165.1)
- added D142: LED, LED_THT:LED_D5.0mm, F.Cu at (452.1, 165.1)
- added D143: LED, LED_THT:LED_D5.0mm, F.Cu at (461.0, 165.1)
- added D144: LED, LED_THT:LED_D5.0mm, F.Cu at (469.9, 165.1)
- added D145: LED, LED_THT:LED_D5.0mm, F.Cu at (475.0, 171.4)
- added D146: LED, LED_THT:LED_D5.0mm, F.Cu at (473.7, 180.3)
- added D147: LED, LED_THT:LED_D5.0mm, F.Cu at (472.4, 189.2)
- added D148: LED, LED_THT:LED_D5.0mm, F.Cu at (471.2, 198.1)
- added D149: LED, LED_THT:LED_D5.0mm, F.Cu at (471.2, 210.8)
- added D15: LED, LED_THT:LED_D5.0mm, F.Cu at (160.0, 241.3)
- added D150: LED, LED_THT:LED_D5.0mm, F.Cu at (469.9, 219.7)
- added D151: LED, LED_THT:LED_D5.0mm, F.Cu at (468.6, 228.6)
- added D152: LED, LED_THT:LED_D5.0mm, F.Cu at (467.4, 237.5)
- added D153: LED, LED_THT:LED_D5.0mm, F.Cu at (435.6, 241.3)
- added D154: LED, LED_THT:LED_D5.0mm, F.Cu at (444.5, 241.3)
- added D155: LED, LED_THT:LED_D5.0mm, F.Cu at (453.4, 241.3)
- added D156: LED, LED_THT:LED_D5.0mm, F.Cu at (462.3, 241.3)
- added D157: LED, LED_THT:LED_D5.0mm, F.Cu at (431.8, 210.8)
- added D158: LED, LED_THT:LED_D5.0mm, F.Cu at (430.5, 219.7)
- added D159: LED, LED_THT:LED_D5.0mm, F.Cu at (429.3, 228.6)
- added D16: LED, LED_THT:LED_D5.0mm, F.Cu at (168.9, 241.3)
- added D160: LED, LED_THT:LED_D5.0mm, F.Cu at (428.0, 237.5)
- added D161: LED, LED_THT:LED_D5.0mm, F.Cu at (435.6, 171.5)
- added D162: LED, LED_THT:LED_D5.0mm, F.Cu at (434.3, 180.3)
- added D163: LED, LED_THT:LED_D5.0mm, F.Cu at (433.1, 189.2)
- added D164: LED, LED_THT:LED_D5.0mm, F.Cu at (431.8, 198.1)
- added D165: LED, LED_THT:LED_D5.0mm, F.Cu at (439.4, 203.2)
- added D166: LED, LED_THT:LED_D5.0mm, F.Cu at (448.3, 203.2)
- added D167: LED, LED_THT:LED_D5.0mm, F.Cu at (457.2, 203.2)
- added D168: LED, LED_THT:LED_D5.0mm, F.Cu at (466.1, 203.2)
- added D169: LED, LED_THT:LED_D5.0mm, F.Cu at (364.5, 221.0)
- added D17: LED, LED_THT:LED_D5.0mm, F.Cu at (138.4, 210.8)
- added D170: LED, LED_THT:LED_D5.0mm, F.Cu at (364.5, 182.9)
- added D171: LED, LED_THT:LED_D5.0mm, F.Cu at (245.1, 185.4)
- added D172: LED, LED_THT:LED_D5.0mm, F.Cu at (245.1, 223.5)
- added D18: LED, LED_THT:LED_D5.0mm, F.Cu at (137.2, 219.7)
- added D19: LED, LED_THT:LED_D5.0mm, F.Cu at (135.9, 228.6)
- added D2: LED, LED_THT:LED_D5.0mm, F.Cu at (158.8, 165.1)
- added D20: LED, LED_THT:LED_D5.0mm, F.Cu at (134.6, 237.5)
- added D21: LED, LED_THT:LED_D5.0mm, F.Cu at (142.2, 171.4)
- added D22: LED, LED_THT:LED_D5.0mm, F.Cu at (141.0, 180.3)
- added D23: LED, LED_THT:LED_D5.0mm, F.Cu at (139.7, 189.2)
- added D24: LED, LED_THT:LED_D5.0mm, F.Cu at (138.4, 198.1)
- added D25: LED, LED_THT:LED_D5.0mm, F.Cu at (146.1, 203.2)
- added D26: LED, LED_THT:LED_D5.0mm, F.Cu at (154.9, 203.2)
- added D27: LED, LED_THT:LED_D5.0mm, F.Cu at (163.8, 203.2)
- added D28: LED, LED_THT:LED_D5.0mm, F.Cu at (172.7, 203.2)
- added D29: LED, LED_THT:LED_D5.0mm, F.Cu at (201.9, 165.1)
- added D3: LED, LED_THT:LED_D5.0mm, F.Cu at (167.6, 165.1)
- added D30: LED, LED_THT:LED_D5.0mm, F.Cu at (210.8, 165.1)
- added D31: LED, LED_THT:LED_D5.0mm, F.Cu at (219.7, 165.1)
- added D32: LED, LED_THT:LED_D5.0mm, F.Cu at (228.6, 165.1)
- added D33: LED, LED_THT:LED_D5.0mm, F.Cu at (233.7, 171.4)
- added D34: LED, LED_THT:LED_D5.0mm, F.Cu at (232.4, 180.3)
- added D35: LED, LED_THT:LED_D5.0mm, F.Cu at (231.1, 189.2)
- added D36: LED, LED_THT:LED_D5.0mm, F.Cu at (229.9, 198.1)
- added D37: LED, LED_THT:LED_D5.0mm, F.Cu at (229.9, 210.8)
- added D38: LED, LED_THT:LED_D5.0mm, F.Cu at (228.6, 219.7)
- added D39: LED, LED_THT:LED_D5.0mm, F.Cu at (227.3, 228.6)
- added D4: LED, LED_THT:LED_D5.0mm, F.Cu at (176.5, 165.1)
- added D40: LED, LED_THT:LED_D5.0mm, F.Cu at (226.1, 237.5)
- added D41: LED, LED_THT:LED_D5.0mm, F.Cu at (194.3, 241.3)
- added D42: LED, LED_THT:LED_D5.0mm, F.Cu at (203.2, 241.3)
- added D43: LED, LED_THT:LED_D5.0mm, F.Cu at (212.1, 241.3)
- added D44: LED, LED_THT:LED_D5.0mm, F.Cu at (221.0, 241.3)
- added D45: LED, LED_THT:LED_D5.0mm, F.Cu at (190.5, 210.8)
- added D46: LED, LED_THT:LED_D5.0mm, F.Cu at (189.2, 219.7)
- added D47: LED, LED_THT:LED_D5.0mm, F.Cu at (188.0, 228.6)
- added D48: LED, LED_THT:LED_D5.0mm, F.Cu at (186.7, 237.5)
- added D49: LED, LED_THT:LED_D5.0mm, F.Cu at (194.3, 171.4)
- added D5: LED, LED_THT:LED_D5.0mm, F.Cu at (181.6, 171.4)
- added D50: LED, LED_THT:LED_D5.0mm, F.Cu at (193.0, 180.3)
- added D51: LED, LED_THT:LED_D5.0mm, F.Cu at (191.8, 189.2)
- added D52: LED, LED_THT:LED_D5.0mm, F.Cu at (190.5, 198.1)
- added D53: LED, LED_THT:LED_D5.0mm, F.Cu at (198.1, 203.2)
- added D54: LED, LED_THT:LED_D5.0mm, F.Cu at (206.9, 203.2)
- added D55: LED, LED_THT:LED_D5.0mm, F.Cu at (215.9, 203.2)
- added D56: LED, LED_THT:LED_D5.0mm, F.Cu at (224.8, 203.2)
- added D57: LED, LED_THT:LED_D5.0mm, F.Cu at (270.5, 165.1)
- added D58: LED, LED_THT:LED_D5.0mm, F.Cu at (279.4, 165.1)
- added D59: LED, LED_THT:LED_D5.0mm, F.Cu at (288.3, 165.1)
- added D6: LED, LED_THT:LED_D5.0mm, F.Cu at (180.3, 180.3)
- added D60: LED, LED_THT:LED_D5.0mm, F.Cu at (297.2, 165.1)
- added D61: LED, LED_THT:LED_D5.0mm, F.Cu at (302.3, 171.4)
- added D62: LED, LED_THT:LED_D5.0mm, F.Cu at (301.0, 180.3)
- added D63: LED, LED_THT:LED_D5.0mm, F.Cu at (299.7, 189.2)
- added D64: LED, LED_THT:LED_D5.0mm, F.Cu at (298.4, 198.1)
- added D65: LED, LED_THT:LED_D5.0mm, F.Cu at (298.4, 210.8)
- added D66: LED, LED_THT:LED_D5.0mm, F.Cu at (297.2, 219.7)
- added D67: LED, LED_THT:LED_D5.0mm, F.Cu at (295.9, 228.6)
- added D68: LED, LED_THT:LED_D5.0mm, F.Cu at (294.6, 237.5)
- added D69: LED, LED_THT:LED_D5.0mm, F.Cu at (262.9, 241.3)
- added D7: LED, LED_THT:LED_D5.0mm, F.Cu at (179.1, 189.2)
- added D70: LED, LED_THT:LED_D5.0mm, F.Cu at (271.8, 241.3)
- added D71: LED, LED_THT:LED_D5.0mm, F.Cu at (280.7, 241.3)
- added D72: LED, LED_THT:LED_D5.0mm, F.Cu at (289.6, 241.3)
- added D73: LED, LED_THT:LED_D5.0mm, F.Cu at (259.1, 210.8)
- added D74: LED, LED_THT:LED_D5.0mm, F.Cu at (257.8, 219.7)
- added D75: LED, LED_THT:LED_D5.0mm, F.Cu at (256.5, 228.6)
- added D76: LED, LED_THT:LED_D5.0mm, F.Cu at (255.3, 237.5)
- added D77: LED, LED_THT:LED_D5.0mm, F.Cu at (262.9, 171.4)
- added D78: LED, LED_THT:LED_D5.0mm, F.Cu at (261.6, 180.3)
- added D79: LED, LED_THT:LED_D5.0mm, F.Cu at (260.4, 189.2)
- added D8: LED, LED_THT:LED_D5.0mm, F.Cu at (177.8, 198.1)
- added D80: LED, LED_THT:LED_D5.0mm, F.Cu at (259.1, 198.1)
- added D81: LED, LED_THT:LED_D5.0mm, F.Cu at (266.7, 203.2)
- added D82: LED, LED_THT:LED_D5.0mm, F.Cu at (275.6, 203.2)
- added D83: LED, LED_THT:LED_D5.0mm, F.Cu at (284.5, 203.2)
- added D84: LED, LED_THT:LED_D5.0mm, F.Cu at (293.4, 203.2)
- added D85: LED, LED_THT:LED_D5.0mm, F.Cu at (322.6, 165.1)
- added D86: LED, LED_THT:LED_D5.0mm, F.Cu at (331.5, 165.1)
- added D87: LED, LED_THT:LED_D5.0mm, F.Cu at (340.4, 165.1)
- added D88: LED, LED_THT:LED_D5.0mm, F.Cu at (349.2, 165.1)
- added D89: LED, LED_THT:LED_D5.0mm, F.Cu at (354.3, 171.4)
- added D9: LED, LED_THT:LED_D5.0mm, F.Cu at (177.8, 210.8)
- added D90: LED, LED_THT:LED_D5.0mm, F.Cu at (353.1, 180.3)
- added D91: LED, LED_THT:LED_D5.0mm, F.Cu at (351.8, 189.2)
- added D92: LED, LED_THT:LED_D5.0mm, F.Cu at (350.5, 198.1)
- added D93: LED, LED_THT:LED_D5.0mm, F.Cu at (350.5, 210.8)
- added D94: LED, LED_THT:LED_D5.0mm, F.Cu at (349.2, 219.7)
- added D95: LED, LED_THT:LED_D5.0mm, F.Cu at (348.0, 228.6)
- added D96: LED, LED_THT:LED_D5.0mm, F.Cu at (346.7, 237.5)
- added D97: LED, LED_THT:LED_D5.0mm, F.Cu at (315.0, 241.3)
- added D98: LED, LED_THT:LED_D5.0mm, F.Cu at (323.9, 241.3)
- added D99: LED, LED_THT:LED_D5.0mm, F.Cu at (332.7, 241.3)
- added Q1: BSS138, Package_TO_SOT_SMD:SOT-23, F.Cu at (128.1, 356.6)
- added Q10: BSS138, Package_TO_SOT_SMD:SOT-23, F.Cu at (133.0, 361.2)
- added Q11: BSS138, Package_TO_SOT_SMD:SOT-23, F.Cu at (133.0, 365.8)
- added Q12: BSS138, Package_TO_SOT_SMD:SOT-23, F.Cu at (133.0, 370.4)
- added Q13: BSS138, Package_TO_SOT_SMD:SOT-23, F.Cu at (133.0, 375.1)
- added Q14: BSS138, Package_TO_SOT_SMD:SOT-23, F.Cu at (133.0, 379.7)
- added Q15: BSS138, Package_TO_SOT_SMD:SOT-23, F.Cu at (133.0, 384.3)
- added Q16: BSS138, Package_TO_SOT_SMD:SOT-23, F.Cu at (133.0, 388.9)
- added Q17: BSS138, Package_TO_SOT_SMD:SOT-23, F.Cu at (137.9, 356.6)
- added Q18: BSS138, Package_TO_SOT_SMD:SOT-23, F.Cu at (137.9, 361.2)
- added Q19: BSS138, Package_TO_SOT_SMD:SOT-23, F.Cu at (137.9, 365.8)
- added Q2: BSS138, Package_TO_SOT_SMD:SOT-23, F.Cu at (128.1, 361.2)
- added Q20: BSS138, Package_TO_SOT_SMD:SOT-23, F.Cu at (137.9, 370.4)
- added Q21: BSS138, Package_TO_SOT_SMD:SOT-23, F.Cu at (137.9, 375.1)
- added Q22: BSS138, Package_TO_SOT_SMD:SOT-23, F.Cu at (137.9, 379.7)
- added Q23: BSS138, Package_TO_SOT_SMD:SOT-23, F.Cu at (137.9, 384.3)
- added Q24: BSS138, Package_TO_SOT_SMD:SOT-23, F.Cu at (137.9, 388.9)
- added Q25: BSS138, Package_TO_SOT_SMD:SOT-23, F.Cu at (142.8, 356.6)
- added Q26: BSS138, Package_TO_SOT_SMD:SOT-23, F.Cu at (142.8, 361.2)
- added Q27: BSS138, Package_TO_SOT_SMD:SOT-23, F.Cu at (142.8, 365.8)
- added Q28: BSS138, Package_TO_SOT_SMD:SOT-23, F.Cu at (142.8, 370.4)
- added Q29: BSS138, Package_TO_SOT_SMD:SOT-23, F.Cu at (142.8, 375.1)
- added Q3: BSS138, Package_TO_SOT_SMD:SOT-23, F.Cu at (128.1, 365.8)
- added Q30: BSS138, Package_TO_SOT_SMD:SOT-23, F.Cu at (142.8, 379.7)
- added Q31: BSS138, Package_TO_SOT_SMD:SOT-23, F.Cu at (142.8, 384.3)
- added Q32: BSS138, Package_TO_SOT_SMD:SOT-23, F.Cu at (142.8, 388.9)
- added Q33: BSS138, Package_TO_SOT_SMD:SOT-23, F.Cu at (147.7, 356.6)
- added Q34: BSS138, Package_TO_SOT_SMD:SOT-23, F.Cu at (147.7, 361.2)
- added Q35: BSS138, Package_TO_SOT_SMD:SOT-23, F.Cu at (147.7, 365.8)
- added Q36: BSS138, Package_TO_SOT_SMD:SOT-23, F.Cu at (147.7, 370.4)
- added Q37: BSS138, Package_TO_SOT_SMD:SOT-23, F.Cu at (147.7, 375.1)
- added Q38: BSS138, Package_TO_SOT_SMD:SOT-23, F.Cu at (147.7, 379.7)
- added Q39: BSS138, Package_TO_SOT_SMD:SOT-23, F.Cu at (147.7, 384.3)
- added Q4: BSS138, Package_TO_SOT_SMD:SOT-23, F.Cu at (128.1, 370.4)
- added Q40: BSS138, Package_TO_SOT_SMD:SOT-23, F.Cu at (147.7, 388.9)
- added Q41: BSS138, Package_TO_SOT_SMD:SOT-23, F.Cu at (152.6, 356.6)
- added Q42: BSS138, Package_TO_SOT_SMD:SOT-23, F.Cu at (152.6, 361.2)
- added Q43: BSS138, Package_TO_SOT_SMD:SOT-23, F.Cu at (245.1, 229.9)
- added Q5: BSS138, Package_TO_SOT_SMD:SOT-23, F.Cu at (128.1, 375.1)
- added Q6: BSS138, Package_TO_SOT_SMD:SOT-23, F.Cu at (128.1, 379.7)
- added Q7: BSS138, Package_TO_SOT_SMD:SOT-23, F.Cu at (128.1, 384.3)
- added Q8: BSS138, Package_TO_SOT_SMD:SOT-23, F.Cu at (128.1, 388.9)
- added Q9: BSS138, Package_TO_SOT_SMD:SOT-23, F.Cu at (133.0, 356.6)
- added R1: 10, Resistor_SMD:R_0603_1608Metric, F.Cu at (142.9, 164.3)
- added R10: 10, Resistor_SMD:R_0603_1608Metric, F.Cu at (229.9, 203.2)
- added R11: 10, Resistor_SMD:R_0603_1608Metric, F.Cu at (186.7, 241.3)
- added R12: 10, Resistor_SMD:R_0603_1608Metric, F.Cu at (190.5, 204.0)
- added R13: 10, Resistor_SMD:R_0603_1608Metric, F.Cu at (193.5, 164.3)
- added R14: 10, Resistor_SMD:R_0603_1608Metric, F.Cu at (190.5, 202.4)
- added R15: 10, Resistor_SMD:R_0603_1608Metric, F.Cu at (263.7, 164.3)
- added R16: 10, Resistor_SMD:R_0603_1608Metric, F.Cu at (302.3, 164.3)
- added R17: 10, Resistor_SMD:R_0603_1608Metric, F.Cu at (298.4, 203.2)
- added R18: 10, Resistor_SMD:R_0603_1608Metric, F.Cu at (255.3, 241.3)
- added R19: 10, Resistor_SMD:R_0603_1608Metric, F.Cu at (259.1, 204.0)
- added R2: 10, Resistor_SMD:R_0603_1608Metric, F.Cu at (181.6, 164.3)
- added R20: 10, Resistor_SMD:R_0603_1608Metric, F.Cu at (262.1, 164.3)
- added R21: 10, Resistor_SMD:R_0603_1608Metric, F.Cu at (259.1, 202.4)
- added R22: 10, Resistor_SMD:R_0603_1608Metric, F.Cu at (315.7, 164.3)
- added R23: 10, Resistor_SMD:R_0603_1608Metric, F.Cu at (354.3, 164.1)
- added R24: 10, Resistor_SMD:R_0603_1608Metric, F.Cu at (350.5, 203.2)
- added R25: 10, Resistor_SMD:R_0603_1608Metric, F.Cu at (307.3, 241.3)
- added R26: 10, Resistor_SMD:R_0603_1608Metric, F.Cu at (311.1, 204.0)
- added R27: 10, Resistor_SMD:R_0603_1608Metric, F.Cu at (314.2, 164.3)
- added R28: 10, Resistor_SMD:R_0603_1608Metric, F.Cu at (311.1, 202.4)
- added R29: 10, Resistor_SMD:R_0603_1608Metric, F.Cu at (384.3, 164.3)
- added R3: 10, Resistor_SMD:R_0603_1608Metric, F.Cu at (177.8, 203.2)
- added R30: 10, Resistor_SMD:R_0603_1608Metric, F.Cu at (422.9, 164.1)
- added R31: 10, Resistor_SMD:R_0603_1608Metric, F.Cu at (419.1, 203.2)
- added R32: 10, Resistor_SMD:R_0603_1608Metric, F.Cu at (375.7, 241.3)
- added R33: 10, Resistor_SMD:R_0603_1608Metric, F.Cu at (379.7, 204.0)
- added R34: 10, Resistor_SMD:R_0603_1608Metric, F.Cu at (382.8, 164.3)
- added R35: 10, Resistor_SMD:R_0603_1608Metric, F.Cu at (379.7, 202.4)
- added R36: 10, Resistor_SMD:R_0603_1608Metric, F.Cu at (436.4, 164.3)
- added R37: 10, Resistor_SMD:R_0603_1608Metric, F.Cu at (475.0, 164.1)
- added R38: 10, Resistor_SMD:R_0603_1608Metric, F.Cu at (471.2, 203.2)
- added R39: 10, Resistor_SMD:R_0603_1608Metric, F.Cu at (428.0, 241.3)
- added R4: 10, Resistor_SMD:R_0603_1608Metric, F.Cu at (134.4, 241.3)
- added R40: 10, Resistor_SMD:R_0603_1608Metric, F.Cu at (431.8, 204.0)
- added R41: 10, Resistor_SMD:R_0603_1608Metric, F.Cu at (434.8, 164.3)
- added R42: 10, Resistor_SMD:R_0603_1608Metric, F.Cu at (431.8, 202.4)
- added R43: 10, Resistor_SMD:R_0603_1608Metric, F.Cu at (364.5, 229.9)
- added R5: 10, Resistor_SMD:R_0603_1608Metric, F.Cu at (138.4, 204.0)
- added R6: 10, Resistor_SMD:R_0603_1608Metric, F.Cu at (141.4, 164.3)
- added R7: 10, Resistor_SMD:R_0603_1608Metric, F.Cu at (138.4, 202.4)
- added R8: 10, Resistor_SMD:R_0603_1608Metric, F.Cu at (195.1, 164.3)
- added R9: 10, Resistor_SMD:R_0603_1608Metric, F.Cu at (233.7, 164.6)
- added U3: 74HC595, Package_SO:SOIC-16_3.9x9.9mm_P1.27mm, F.Cu at (156.2, 228.6)
- added U4: 74HC595, Package_SO:SOIC-16_3.9x9.9mm_P1.27mm, F.Cu at (208.3, 228.6)
- added U5: 74HC595, Package_SO:SOIC-16_3.9x9.9mm_P1.27mm, F.Cu at (276.9, 228.6)
- added U6: 74HC595, Package_SO:SOIC-16_3.9x9.9mm_P1.27mm, F.Cu at (328.9, 228.6)
- added U7: 74HC595, Package_SO:SOIC-16_3.9x9.9mm_P1.27mm, F.Cu at (397.5, 228.6)
- added U8: 74HC595, Package_SO:SOIC-16_3.9x9.9mm_P1.27mm, F.Cu at (449.6, 228.6)
Connections:
- U1 pad 14: unconnected-(U1-G12-Pad14) -> Net-(Q43-G)
- U1 pad 19: unconnected-(U1-G39-Pad19) -> /SRCLK
- U1 pad 21: unconnected-(U1-G40-Pad21) -> /OE
- U1 pad 23: unconnected-(U1-G41-Pad23) -> /RCLK
- U1 pad 25: unconnected-(U1-G42-Pad25) -> /SRCLR
- U1 pad 27: unconnected-(U1-G46-Pad27) -> /SER

Commit message: 配線した
Parts:
- moved Q36 353.0 mm to (464.6, 214.9), turned to 90 degrees
- moved Q37 350.8 mm to (459.7, 214.9), turned to 90 degrees
- moved Q38 348.6 mm to (454.9, 214.9), turned to 90 degrees
- moved Q39 346.6 mm to (450.1, 214.9), turned to 90 degrees
- moved Q40 344.7 mm to (445.3, 214.9), turned to 90 degrees
- moved Q41 320.8 mm to (440.4, 214.9), turned to 90 degrees
- moved Q42 318.6 mm to (435.6, 214.9), turned to 90 degrees
- moved Q29 313.6 mm to (412.5, 215.0), turned to 90 degrees
- moved Q30 311.9 mm to (407.7, 215.0), turned to 90 degrees
- moved Q31 310.3 mm to (402.8, 215.0), turned to 90 degrees
- moved Q32 308.9 mm to (398.0, 215.0), turned to 90 degrees
- moved Q33 283.4 mm to (393.2, 215.0), turned to 90 degrees
- moved Q34 281.6 mm to (388.4, 215.0), turned to 90 degrees
- moved Q35 280.0 mm to (383.5, 214.9), turned to 90 degrees
- moved Q22 264.0 mm to (344.2, 214.9), turned to 90 degrees
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Routing:
- net /OE: track 0.00 -> 360.8 mm, vias 0 -> 6
- net /RCLK: track 0.00 -> 353.9 mm, vias 0 -> 6
- net /SER: track 0.00 -> 347.4 mm, vias 0 -> 6
- net /SRCLR: track 0.00 -> 346.2 mm, vias 0 -> 6
- net Net-(D170-K): track 0.00 -> 122.5 mm
- net Net-(U6-QH'): track 0.00 -> 83.7 mm, vias 0 -> 2
- net Net-(U4-QH'): track 0.00 -> 83.7 mm, vias 0 -> 2
- net Net-(U5-QH'): track 0.00 -> 67.2 mm, vias 0 -> 2
- net Net-(U3-QH'): track 0.00 -> 67.2 mm, vias 0 -> 2
- net Net-(U7-QH'): track 0.00 -> 67.1 mm, vias 0 -> 2
- net Net-(D116-K): track 0.00 -> 51.1 mm, vias 0 -> 1
- net Net-(D144-K): track 0.00 -> 51.1 mm, vias 0 -> 1
- net Net-(D4-K): track 0.00 -> 51.0 mm, vias 0 -> 1
- net Net-(D88-K): track 0.00 -> 51.0 mm, vias 0 -> 1
- net Net-(D60-K): track 0.00 -> 51.0 mm, vias 0 -> 1
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- added copper zone on B.Cu, net GND

Commit message: 仕上げた
Parts:
- added C1: 0.22u, Capacitor_SMD:C_0603_1608Metric, F.Cu at (107.4, 201.4)
- added C2: 0.1u, Capacitor_SMD:C_0603_1608Metric, F.Cu at (107.4, 212.6)
- added D173: D, Diode_SMD:D_SOD-523, F.Cu at (101.6, 207.0)
- added J1: Barrel_Jack_Switch, Connector_BarrelJack:BarrelJack_Horizontal, B.Cu at (121.9, 196.4)
- added U9: L7805, Package_TO_SOT_SMD:TO-252-2, F.Cu at (110.5, 207.0)
Routing:
- net Net-(Q43-G): track 0.00 -> 152.5 mm
- net +3.3V: track 0.00 -> 50.7 mm
- net +12V: track 0.00 -> 26.6 mm
- net +5V: track 0.00 -> 5.07 mm
- net GND: track 46.8 -> 48.8 mm, vias 43 -> 48
- added copper zone on F.Cu, net +5V
