File: 2U-NTP-Clock.kicad_sch (KiCad schematic)
At the start: 277 parts, among them J1 Barrel_Jack_Switch, Q1 BSS138, Q10 BSS138, Q11 BSS138, Q12 BSS138, Q13 BSS138, Q14 BSS138, Q15 BSS138, Q16 BSS138, Q17 BSS138, Q18 BSS138, Q19 BSS138, Q2 BSS138, Q20 BSS138, Q21 BSS138, Q22 BSS138, Q23 BSS138, Q24 BSS138, Q25 BSS138, Q26 BSS138, Q27 BSS138, Q28 BSS138, Q29 BSS138, Q3 BSS138, Q30 BSS138, Q31 BSS138, Q32 BSS138, Q33 BSS138, Q34 BSS138, Q35 BSS138, Q36 BSS138, Q37 BSS138, Q38 BSS138, Q39 BSS138, Q4 BSS138, Q40 BSS138, Q41 BSS138, Q42 BSS138, Q43 BSS138, Q5 BSS138, Q6 BSS138, Q7 BSS138, Q8 BSS138, Q9 BSS138, SW1 SW_Push, SW2 SW_Push, SW3 SW_Push, SW4 SW_Push, SW5 SW_Push, SW6 SW_Slide_DPDT, U3 74HC595, U4 74HC595, U5 74HC595, U6 74HC595, U7 74HC595, U8 74HC595, U9 L7805

Commit message: デバッグポート・Eth PHY の実装
Parts:
- added J2: Conn_01x06_Socket, symbol Connector:Conn_01x06_Socket
- added U10: ~, symbol eth:wiz850io
Connections:
- net +3.3V: now also J2.1 (Pin_1), U10.10 (3.3V), U10.11 (3.3V)
- net GND: now also J2.6 (Pin_6), U10.1 (GND), U10.2 (GND)
- net CS: now reaches U1.10 (G10)
- net CS: now also U10.5 (SCNn)
- net MOSI: now reaches U1.12 (G11)
- net MOSI: now also U10.3 (MOSI)
- net at Q43.1 (G): now also U1.6 (G6); no longer U1.14 (G12)
- net BOOT-G0: now reaches U1.20 (G0/Boot)
- net BOOT-G0: now also J2.5 (Pin_5)
- net RST-EN: now reaches U1.22 (EN)
- net RST-EN: now also J2.4 (Pin_4)
- net TX-RX0: now reaches U1.24 (G44/RX)
- net TX-RX0: now also J2.3 (Pin_3)
- net RX-TX0: now reaches U1.26 (G43/TX)
- net RX-TX0: now also J2.2 (Pin_2)
- net DETECT: now reaches U1.7 (G7)
- net DETECT: now also U10.12 (GND)
- net RESET: now reaches U1.8 (G8)
- net RESET: now also U10.8 (RSTn)
- net MISO: now reaches U1.9 (G9)
- net MISO: now also U10.7 (MISO)
- new net CLK: U1.14 (G12), U10.4 (SCLK)
- no-connect marks 9 -> 10

Commit message: 追加部品にフットプリント割り当て
Parts:
- J2: footprint (none) -> Connector_PinSocket_2.54mm:PinSocket_1x06_P2.54mm_Vertical
- U10: footprint (none) -> eth:WIZ850io
Changed lines of the file:
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@@
 			)
 		)
-		(property "Footprint" ""
+		(property "Footprint" "Connector_PinSocket_2.54mm:PinSocket_1x06_P2.54mm_Vertical"
 			(at 83.82 44.45 0)
 			(effects
@@
 			)
 		)
-		(property "Footprint" ""
+		(property "Footprint" "eth:WIZ850io"
 			(at 45.72 334.518 0)
 			(effects

Commit message: 部品の割り当てを変更
Parts:
- C2: LCSC C6903803 -> C14663
Changed lines of the file:
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@@
 			)
 		)
-		(property "LCSC" "C6903803"
+		(property "LCSC" "C14663"
 			(at 63.5 182.88 0)
 			(effects

Commit message: 配線修正
Connections:
- net at D46.1 (K): now also D48.1 (K), Q12.3 (D); no longer D47.2 (A)
- net at D9.2 (A), R3.2: now also D11.2 (A)
- net at D107.2 (A): now also D105.2 (A), R27.2; no longer D106.1 (K)
- net at D94.1 (K): now also D96.1 (K), Q24.3 (D); no longer D95.2 (A)
- net at D36.1 (K), Q9.3 (D): now also D34.1 (K)
- net at D6.1 (K): now also D8.1 (K), Q2.3 (D); no longer D7.2 (A)
- net at D126.1 (K): now also D128.1 (K), Q32.3 (D); no longer D127.2 (A)
- net at D37.2 (A), R10.2: now also D39.2 (A)
- net at D59.2 (A): now also D57.2 (A), R15.2; no longer D58.1 (K)
- net at D2.1 (K): now also D4.1 (K), Q1.3 (D); no longer D3.2 (A)
- net at D153.2 (A), R39.2: now also D155.2 (A)
- net at D60.1 (K), Q15.3 (D): now also D58.1 (K)
- net at D118.1 (K): now also D120.1 (K), Q30.3 (D); no longer D119.2 (A)
- net at D159.2 (A): now also D157.2 (A), R40.2; no longer D158.1 (K)
- net at D133.2 (A), R34.2: now also D135.2 (A)
- net at D31.2 (A): now also D29.2 (A), R8.2; no longer D30.1 (K)
- net at D112.1 (K), Q28.3 (D): now also D110.1 (K)
- net at D113.2 (A), R29.2: now also D115.2 (A)
- net at D93.2 (A), R24.2: now also D95.2 (A)
- net at D136.1 (K), Q34.3 (D): now also D134.1 (K)
- net at D123.2 (A): now also D121.2 (A), R31.2; no longer D122.1 (K)
- net at D142.1 (K): now also D144.1 (K), Q36.3 (D); no longer D143.2 (A)
- net at D49.2 (A), R13.2: now also D51.2 (A)
- net at D145.2 (A), R37.2: now also D147.2 (A)
- net at D129.2 (A), R33.2: now also D131.2 (A)
- net at D62.1 (K): now also D64.1 (K), Q16.3 (D); no longer D63.2 (A)
- net at D54.1 (K): now also D56.1 (K), Q14.3 (D); no longer D55.2 (A)
- net at D171.2 (A): now also D169.2 (A), R43.2; no longer D170.1 (K)
- net at D163.2 (A): now also D161.2 (A), R41.2; no longer D162.1 (K)
- net at D80.1 (K), Q20.3 (D): now also D78.1 (K)
- net at D66.1 (K): now also D68.1 (K), Q17.3 (D); no longer D67.2 (A)
- net at D74.1 (K): now also D76.1 (K), Q19.3 (D); no longer D75.2 (A)
- net at D12.1 (K), Q3.3 (D): now also D10.1 (K)
- net at D89.2 (A), R23.2: now also D91.2 (A)
- net at D32.1 (K), Q8.3 (D): now also D30.1 (K)
- net at D45.2 (A), R12.2: now also D47.2 (A)
- net at D141.2 (A), R36.2: now also D143.2 (A)
- net at D50.1 (K): now also D52.1 (K), Q13.3 (D); no longer D51.2 (A)
- net at D79.2 (A): now also D77.2 (A), R20.2; no longer D78.1 (K)
- net at D61.2 (A), R16.2: now also D63.2 (A)
- net at D108.1 (K), Q27.3 (D): now also D106.1 (K)
- net at D109.2 (A), R28.2: now also D111.2 (A)
- net at D156.1 (K), Q39.3 (D): now also D154.1 (K)
- net at D13.2 (A), R4.2: now also D15.2 (A)
- net at D102.1 (K): now also D104.1 (K), Q26.3 (D); no longer D103.2 (A)
- net at D97.2 (A), R25.2: now also D99.2 (A)
- net at D33.2 (A), R9.2: now also D35.2 (A)
- net at D25.2 (A), R7.2: now also D27.2 (A)
- net at D65.2 (A), R17.2: now also D67.2 (A)
- net at D22.1 (K): now also D24.1 (K), Q6.3 (D); no longer D23.2 (A)
- net at D41.2 (A), R11.2: now also D43.2 (A)
- net at D167.2 (A): now also D165.2 (A), R42.2; no longer D166.1 (K)
- net at D42.1 (K): now also D44.1 (K), Q11.3 (D); no longer D43.2 (A)
- net at D73.2 (A), R19.2: now also D75.2 (A)
- net at D40.1 (K), Q10.3 (D): now also D38.1 (K)
- net at D116.1 (K), Q29.3 (D): now also D114.1 (K)
- net at D100.1 (K), Q25.3 (D): now also D98.1 (K)
- net at D85.2 (A), R22.2: now also D87.2 (A)
- net at D130.1 (K): now also D132.1 (K), Q33.3 (D); no longer D131.2 (A)
- net at D81.2 (A), R21.2: now also D83.2 (A)
- net at D18.1 (K): now also D20.1 (K), Q5.3 (D); no longer D19.2 (A)
- net at D86.1 (K): now also D88.1 (K), Q22.3 (D); no longer D87.2 (A)
- net at D1.2 (A), R1.2: now also D3.2 (A)
- net at D21.2 (A), R6.2: now also D23.2 (A)
- net at D72.1 (K), Q18.3 (D): now also D70.1 (K)
- net at D151.2 (A): now also D149.2 (A), R38.2; no longer D150.1 (K)
- net at D137.2 (A), R35.2: now also D139.2 (A)
- net at D160.1 (K), Q40.3 (D): now also D158.1 (K)
- net at D138.1 (K): now also D140.1 (K), Q35.3 (D); no longer D139.2 (A)
- net at D28.1 (K), Q7.3 (D): now also D26.1 (K)
- net at D53.2 (A), R14.2: now also D55.2 (A)
- net at D5.2 (A), R2.2: now also D7.2 (A)
- net at D17.2 (A), R5.2: now also D19.2 (A)
- net at D148.1 (K), Q37.3 (D): now also D146.1 (K)
- net at D14.1 (K): now also D16.1 (K), Q4.3 (D); no longer D15.2 (A)
- net at D71.2 (A): now also D69.2 (A), R18.2; no longer D70.1 (K)
- net at D172.1 (K), Q43.3 (D): now also D170.1 (K)
- net at D124.1 (K), Q31.3 (D): now also D122.1 (K)
- net at D164.1 (K), Q41.3 (D): now also D162.1 (K)
- net at D90.1 (K): now also D92.1 (K), Q23.3 (D); no longer D91.2 (A)
- net at D125.2 (A), R32.2: now also D127.2 (A)
- net at D101.2 (A), R26.2: now also D103.2 (A)
- net at D84.1 (K), Q21.3 (D): now also D82.1 (K)
- net at D117.2 (A), R30.2: now also D119.2 (A)
- net at D152.1 (K), Q38.3 (D): now also D150.1 (K)
- net at D168.1 (K), Q42.3 (D): now also D166.1 (K)
