File: 2U-NTP-Clock.kicad_sch (KiCad schematic)
At the start: 279 parts, among them J1 Barrel_Jack_Switch, J2 Conn_01x06_Socket, Q1 BSS138, Q10 BSS138, Q11 BSS138, Q12 BSS138, Q13 BSS138, Q14 BSS138, Q15 BSS138, Q16 BSS138, Q17 BSS138, Q18 BSS138, Q19 BSS138, Q2 BSS138, Q20 BSS138, Q21 BSS138, Q22 BSS138, Q23 BSS138, Q24 BSS138, Q25 BSS138, Q26 BSS138, Q27 BSS138, Q28 BSS138, Q29 BSS138, Q3 BSS138, Q30 BSS138, Q31 BSS138, Q32 BSS138, Q33 BSS138, Q34 BSS138, Q35 BSS138, Q36 BSS138, Q37 BSS138, Q38 BSS138, Q39 BSS138, Q4 BSS138, Q40 BSS138, Q41 BSS138, Q42 BSS138, Q43 BSS138, Q5 BSS138, Q6 BSS138, Q7 BSS138, Q8 BSS138, Q9 BSS138, SW1 SW_Push, SW2 SW_Push, SW3 SW_Push, SW4 SW_Push, SW5 SW_Push, SW6 SW_Slide_DPDT, U3 74HC595, U4 74HC595, U5 74HC595, U6 74HC595, U7 74HC595, U8 74HC595, U9 L7805

Commit message: 破綻箇所修正
Connections:
- net at Q9.3 (D): now also D34.1 (K), D36.1 (K)
- net at D59.2 (A): now also D57.2 (A), R15.2
- net at D2.1 (K): now also D4.1 (K), Q1.3 (D)
- net at D106.1 (K): now also D108.1 (K), Q27.3 (D)
- net at D60.1 (K), Q15.3 (D): now also D58.1 (K)
- net at D118.1 (K): now also D120.1 (K), Q30.3 (D)
- net at D119.2 (A): now also D117.2 (A), R30.2
- net at D133.2 (A), R34.2: now also D135.2 (A)
- net at D3.2 (A): now also D1.2 (A), R1.2
- net at D112.1 (K), Q28.3 (D): now also D110.1 (K)
- net at D113.2 (A), R29.2: now also D115.2 (A)
- net at D93.2 (A), R24.2: now also D95.2 (A)
- net at D123.2 (A), R31.2: now also D121.2 (A)
- net at D49.2 (A), R13.2: now also D51.2 (A)
- net at D145.2 (A), R37.2: now also D147.2 (A)
- net at D62.1 (K): now also D64.1 (K), Q16.3 (D)
- net at D54.1 (K): now also D56.1 (K), Q14.3 (D)
- net at D122.1 (K): now also D124.1 (K), Q31.3 (D)
- net at Q20.3 (D): now also D78.1 (K), D80.1 (K)
- net at D66.1 (K), D68.1 (K): now also Q17.3 (D)
- net at D74.1 (K): now also D76.1 (K), Q19.3 (D)
- net at D12.1 (K), Q3.3 (D): now also D10.1 (K)
- net at D32.1 (K), Q8.3 (D): now also D30.1 (K)
- net at D45.2 (A), R12.2: now also D47.2 (A)
- net at D141.2 (A), R36.2: now also D143.2 (A)
- net at D79.2 (A): now also D77.2 (A), R20.2
- net at D52.1 (K), Q13.3 (D): now also D50.1 (K)
- net at D109.2 (A), R28.2: now also D111.2 (A)
- net at D67.2 (A): now also D65.2 (A), R17.2
- net at D13.2 (A), D15.2 (A), R4.2: no longer D14.1 (K)
- net at D102.1 (K), D104.1 (K), Q26.3 (D): no longer D103.2 (A)
- net at D33.2 (A): now also D35.2 (A), R9.2
- net at R7.2: now also D25.2 (A), D27.2 (A)
- net at D22.1 (K): now also D24.1 (K), Q6.3 (D)
- net at D41.2 (A), R11.2: now also D43.2 (A)
- net at D167.2 (A): now also D165.2 (A), R42.2
- net at D42.1 (K): now also D44.1 (K), Q11.3 (D)
- net at D40.1 (K), Q10.3 (D): now also D38.1 (K)
- net at D116.1 (K), Q29.3 (D): now also D114.1 (K)
- net at D100.1 (K), Q25.3 (D): now also D98.1 (K)
- net at D85.2 (A), D87.2 (A), R22.2: no longer D86.1 (K), D88.1 (K), Q22.3 (D)
- net at D18.1 (K): now also D20.1 (K), Q5.3 (D)
- net at D72.1 (K), Q18.3 (D): now also D70.1 (K)
- net at D151.2 (A): now also D149.2 (A), R38.2
- net at D19.2 (A): now also D17.2 (A), R5.2
- net at D132.1 (K), Q33.3 (D): now also D130.1 (K)
- net at D158.1 (K), D160.1 (K): now also Q40.3 (D)
- net at D28.1 (K), Q7.3 (D): now also D26.1 (K)
- net at D53.2 (A): now also D55.2 (A), R14.2
- net at D5.2 (A), R2.2: now also D7.2 (A)
- net at D148.1 (K), Q37.3 (D): now also D146.1 (K)
- net at D172.1 (K), Q43.3 (D): now also D170.1 (K)
- net at D140.1 (K), Q35.3 (D): now also D138.1 (K)
- net at D164.1 (K), Q41.3 (D): now also D162.1 (K)
- net at D125.2 (A), R32.2: now also D127.2 (A)
- net at D101.2 (A), R26.2: now also D103.2 (A)
- net at D150.1 (K): now also D152.1 (K), Q38.3 (D)
- net at D16.1 (K), Q4.3 (D): now also D14.1 (K)
- new net: D86.1 (K), D88.1 (K), Q22.3 (D)

Commit message: MOSFET のプルダウン抵抗を追加
Parts:
- added R44, R45, R46, R47, R48, R49, R50, R51, R52, R53, R54, R55, R56, R57, R58, R59, R60, R61, R62, R63, R64, R65, R66, R67, R68, R69, R70, R71, R72, R73, R74, R75, R76, R77, R78, R79, R80, R81, R82, R83, R84, R85, R86: 100k, Resistor_SMD:R_0603_1608Metric, symbol Device:R
Connections:
- net GND: now also R44.2, R45.2, R46.2, R47.2, R48.2, R49.2, R50.2, R51.2, R52.2, R53.2, R54.2, R55.2, R56.2, R57.2, R58.2, R59.2, R60.2, R61.2, R62.2, R63.2, R64.2, R65.2, R66.2, R67.2, R68.2, R69.2, R70.2, R71.2, R72.2, R73.2, R74.2, R75.2, R76.2, R77.2, R78.2, R79.2, R80.2, R81.2, R82.2, R83.2, R84.2, R85.2, R86.2
- net at Q9.1 (G), U4.2 (QC): now also R52.1
- net at Q30.1 (G), U7.2 (QC): now also R73.1
- net at Q15.1 (G), U5.1 (QB): now also R58.1
- net at Q16.1 (G), U5.2 (QC): now also R59.1
- net at Q17.1 (G), U5.3 (QD): now also R60.1
- net at Q18.1 (G), U5.4 (QE): now also R61.1
- net at Q19.1 (G), U5.5 (QF): now also R62.1
- net at Q20.1 (G), U5.6 (QG): now also R63.1
- net at Q21.1 (G), U5.7 (QH): now also R64.1
- net at Q32.1 (G), U7.4 (QE): now also R75.1
- net at Q14.1 (G), U4.7 (QH): now also R57.1
- net at Q27.1 (G), U6.6 (QG): now also R70.1
- net at Q13.1 (G), U4.6 (QG): now also R56.1
- net at Q43.1 (G), U1.6 (G6): now also R86.1
- net at Q39.1 (G), U8.4 (QE): now also R82.1
- net at Q8.1 (G), U4.1 (QB): now also R51.1
- net at Q12.1 (G), U4.5 (QF): now also R55.1
- net at Q36.1 (G), U8.1 (QB): now also R79.1
- net at Q37.1 (G), U8.2 (QC): now also R80.1
- net at Q38.1 (G), U8.3 (QD): now also R81.1
- net at Q40.1 (G), U8.5 (QF): now also R83.1
- net at Q41.1 (G), U8.6 (QG): now also R84.1
- net at Q42.1 (G), U8.7 (QH): now also R85.1
- net at Q25.1 (G), U6.4 (QE): now also R68.1
- net at Q11.1 (G), U4.4 (QE): now also R54.1
- net at Q3.1 (G), U3.3 (QD): now also R46.1
- net at Q22.1 (G), U6.1 (QB): now also R65.1
- net at Q10.1 (G), U4.3 (QD): now also R53.1
- net at Q29.1 (G), U7.1 (QB): now also R72.1
- net at Q31.1 (G), U7.3 (QD): now also R74.1
- net at Q33.1 (G), U7.5 (QF): now also R76.1
- net at Q34.1 (G), U7.6 (QG): now also R77.1
- net at Q35.1 (G), U7.7 (QH): now also R78.1
- net at Q7.1 (G), U3.7 (QH): now also R50.1
- net at Q2.1 (G), U3.2 (QC): now also R45.1
- net at Q28.1 (G), U6.7 (QH): now also R71.1
- net at Q24.1 (G), U6.3 (QD): now also R67.1
- net at Q6.1 (G), U3.6 (QG): now also R49.1
- net at Q1.1 (G), U3.1 (QB): now also R44.1
- net at Q4.1 (G), U3.4 (QE): now also R47.1
- net at Q5.1 (G), U3.5 (QF): now also R48.1
- net at Q23.1 (G), U6.2 (QC): now also R66.1
- net at Q26.1 (G), U6.5 (QF): now also R69.1
